File: eagle/Duck/Controller/controller_v1/v1.sch (EAGLE design)
At the start: 6 parts

Commit message: board design
Parts:
- added R1, R2: (no value), rcl:R-US_0309/12
- U$4, U$5: value PUSH_SW -> PUSH_SW_LED; device Switch:PUSH_SW -> Switch:PUSH_SW_LED
Connections:
- new net 34: R1.1, U$3.34
- new net 35: R2.1, U$3.35
- new net N$1: U$3.TX
- new net N$3: R1.2, U$4.PI
- new net N$4: R2.2, U$5.PI
- net +3V3: now also U$4.P4, U$5.P4; no longer U$4.P3, U$5.P3
- net GND: now also U$4.PO, U$5.PO

Commit message: Upside down
Connections:
- removed net 16: U$3.16, U$4.P1
- removed net 17: U$3.17, U$5.P1
- removed net 34: R1.1, U$3.34
- removed net 35: R2.1, U$3.35
- new net LED1: R1.1, U$3.14
- new net LED2: R2.1, U$3.13
- new net SW1: U$3.35, U$4.P1
- new net SW2: U$3.27, U$5.P1
- net RS: now also U$3.26; no longer U$3.2
- net RST: now also U$3.25; no longer U$3.4
